Commit message: 30/12/24

File: src/bumperbot_description/urdf/bumperbot.urdf.xacro (robot description, xacro)
@@ -1,6 +1,11 @@
 <?xml version="1.0"?>
 <robot xmlns:xacro="http://www.ros.org/wiki/xacro" name="bumperbot">
+    <xacro:arg name="is_ignition" default="true" />
     <link name="base_footprint"/>
     <link name="base_link">
+        <inertial>
+            <origin xyz="0 0 0.04" rpy ="0.0 0.25 0.3" />
+            <mass value="8.2573504e-01" />
+        </inertial>
         <visual>
             <origin rpy="0 0 0" xyz="0 0 0" />
@@ -9,4 +14,10 @@
             </geometry>
         </visual>
+        <collision>
+            <origin rpy="0 0 0" xyz="0 0 0" />
+            <geometry>
+                <mesh filename="package://bumperbot_description/meshes/base_link.STL"/>
+            </geometry>
+        </collision>
     </link>
     <joint name="base_joint" type="fixed">
@@ -22,4 +33,10 @@
             </geometry>
         </visual>
+        <collision>
+            <origin xyz="0 -0.015 0" rpy="1.57 0 0" />
+            <geometry>
+                <sphere radius="0.033" />
+            </geometry>
+        </collision>
     </link>
     <joint name="wheel_right_joint" type ="continuous">
@@ -36,4 +53,10 @@
             </geometry>
         </visual>
+        <collision>
+            <origin xyz="0 0.015 0" rpy="1.57 0 0" />
+            <geometry>
+                <sphere radius="0.033" />
+            </geometry>
+        </collision>
     </link>
     <joint name="wheel_left_joint" type ="continuous">
@@ -50,4 +73,10 @@
             </geometry>
         </visual>
+        <collision>
+            <origin xyz="0 0 0" rpy="0 0 0" />
+            <geometry>
+                <sphere radius="0.005" />
+            </geometry>
+        </collision>
     </link>
      <joint name="caster_front_joint" type ="fixed">
@@ -63,4 +92,10 @@
             </geometry>
         </visual>
+        <collision>
+            <origin xyz="0 0 0" rpy="0 0 0" />
+            <geometry>
+                <sphere radius="0.005" />
+            </geometry>
+        </collision>
     </link>
      <joint name="caster_rear_joint" type ="fixed">
